Commit message: update

File: src/sdvt_description/urdf/cart.urdf.xacro (robot description, xacro)
@@ -1,6 +1,4 @@
 <?xml version="1.0"?>
 <robot name="sdvt_robot" xmlns:xacro="http://ros.org/wiki/xacro">
-  <!-- Included URDF/XACRO Files -->
-  <xacro:include filename="$(find husky_description)/urdf/wheel.urdf.xacro" />
   <property name="M_PI" value="3.14159"/>
   <!-- Base Size -->
@@ -9,11 +7,10 @@
   <property name="base_z_size" value="1.144" />
   <!-- Wheel Mounting Positions -->
-  <xacro:property name="wheelbase" value="1.6" />
-  <xacro:property name="track" value="1.21" />
-  <xacro:property name="wheel_vertical_offset" value="1.3282" />
+  <xacro:property name="wheelbase" value="1.9" />
+  <xacro:property name="track" value="1.2" />
+  <xacro:property name="wheel_vertical_offset" value="0.03282" />
   <!-- Wheel Properties -->
   <xacro:property name="wheel_length" value="0.23" />
   <xacro:property name="wheel_radius" value="0.25" />
-  <xacro:macro name="sdvt_robot">
     <!-- Base link is the center of the robot's bottom plate -->
     <link name="base_link">
@@ -22,5 +19,5 @@
         <geometry>
           <!--<mesh filename="package://sdvt_description/meshes/base_link.dae" />-->
-          <box size="${base_x_size} ${base_y_size} ${base_z_size}"/>
+          <box size="${base_x_size/4} ${base_y_size/4} ${base_z_size/4}"/>
         </geometry>
       </visual>
@@ -68,4 +65,49 @@
     <gazebo reference="imu_link">
     </gazebo>
+    <!-- SDVT wheel xacro -->
+	<xacro:macro name="sdvt_wheel" params="wheel_prefix *joint_pose">
+		<link name="${wheel_prefix}_wheel_link">
+			<inertial>
+				<mass value="2.637" />
+				<origin xyz="0 0 0" />
+				<inertia  ixx="0.02467" ixy="0" ixz="0" iyy="0.02467" iyz="0" izz="0.04411" />
+			</inertial>
+			<visual>
+				<origin xyz="0 0 0" rpy="0 0 0" />
+				<geometry>
+					<!--<mesh filename="package://husky_description/meshes/wheel.dae" />-->
+ 					<cylinder length="${wheel_length/4}" radius="${wheel_radius/4}" />
+				</geometry>
+			</visual>
+			<collision>
+				<origin xyz="0 0 0" rpy="${M_PI/2} 0 0" />
+				<geometry>
+					<cylinder length="${wheel_length}" radius="${wheel_radius}" />
+				</geometry>
+			</collision>
+		</link>
+		<gazebo reference="${wheel_prefix}_wheel_link">
+			<mu1 value="1.0"/>
+			<mu2 value="1.0"/>
+			<kp value="10000000.0" />
+			<kd value="1.0" />
+			<fdir1 value="1 0 0"/>
+		</gazebo>
+		<joint name="${wheel_prefix}_wheel" type="continuous">
+			<parent link="base_link"/>
+			<child link="${wheel_prefix}_wheel_link"/>
+			<xacro:insert_block name="joint_pose"/>
+			<axis xyz="0 1 0" rpy="0 0 0" />
+		</joint>
+		<transmission name="${wheel_prefix}_wheel_trans" type="SimpleTransmission">
+			<type>transmission_interface/SimpleTransmission</type>
+			<actuator name="${wheel_prefix}_wheel_motor">
+				<mechanicalReduction>1</mechanicalReduction>
+			</actuator>
+			<joint name="${wheel_prefix}_wheel">
+				<hardwareInterface>VelocityJointInterface</hardwareInterface>
+			</joint>
+		</transmission>
+	</xacro:macro>
     <!-- SDVT wheel macros -->
     <xacro:sdvt_wheel wheel_prefix="front_left">
@@ -81,5 +123,25 @@
       <origin xyz="${-wheelbase/2} ${-track/2} ${wheel_vertical_offset}" rpy="0 0 0" />
     </xacro:sdvt_wheel>
- <!--   <xacro:sdvt_decorate /> -->
-  </xacro:macro>
+  <!-- Decoration description  <xacro:sdvt_decorate /> -->
+  <!-- Same note as applies to imu_link -->
+  <link name="navsat_link">
+    <visual>
+      <geometry>
+        <cylinder radius="0.026" length="0.016" />
+      </geometry>
+      <origin xyz="0 0 0.008" />
+      <material name="black" />
+    </visual>
+  </link>
+  <joint name="navsat_joint" type="fixed">
+    <parent link="base_link" />
+    <child link="navsat_link" />
+    <origin xyz="-0.180 0.126 0.1815" />
+  </joint>
+  <!-- Left lidar -->
+  <!-- Right lidar -->
+  <!-- Front radar -->
+  <!-- Left camera -->
+  <!-- Right camera -->
+  <xacro:include filename="sdvt.gazebo" />
 </robot>

Commit message: made some changes

File: src/sdvt_description/urdf/cart.urdf.xacro (robot description, xacro)
@@ -3,21 +3,20 @@
   <property name="M_PI" value="3.14159"/>
   <!-- Base Size -->
-  <property name="base_x_size" value="1.978" />
-  <property name="base_y_size" value="1.19" />
-  <property name="base_z_size" value="1.144" />
+  <property name="base_x_size" value="3" />
+  <property name="base_y_size" value="2" />
+  <property name="base_z_size" value="1" />
   <!-- Wheel Mounting Positions -->
-  <xacro:property name="wheelbase" value="1.9" />
-  <xacro:property name="track" value="1.2" />
-  <xacro:property name="wheel_vertical_offset" value="0.03282" />
+  <xacro:property name="wheelbase" value="4.8" />
+  <xacro:property name="track" value="2.63" />
+  <xacro:property name="wheel_vertical_offset" value="-0.5" />
   <!-- Wheel Properties -->
-  <xacro:property name="wheel_length" value="0.23" />
-  <xacro:property name="wheel_radius" value="0.25" />
+  <xacro:property name="wheel_length" value="1" />
+  <xacro:property name="wheel_radius" value="0.24" />
     <!-- Base link is the center of the robot's bottom plate -->
     <link name="base_link">
       <visual>
-        <origin xyz="0 0 0" rpy="0 0 0" />
+        <origin xyz="0 1.65 0" rpy="${M_PI/2} 0 0" />
         <geometry>
-          <!--<mesh filename="package://sdvt_description/meshes/base_link.dae" />-->
-          <box size="${base_x_size/4} ${base_y_size/4} ${base_z_size/4}"/>
+          <mesh filename="package://sdvt_description/meshes/New Frame with car no wheels.stl" scale="0.03 0.03 0.03"/>
         </geometry>
       </visual>
@@ -25,11 +24,5 @@
         <origin xyz="0 0 ${base_z_size/4}" rpy="0 0 0" />
         <geometry>
-          <box size="${base_x_size} ${base_y_size} ${base_z_size/2}"/>
-        </geometry>
-      </collision>
-      <collision>
-        <origin xyz="0 0 ${base_z_size*3/4}" rpy="0 0 0" />
-        <geometry>
-          <box size="${base_x_size*4/5} ${base_y_size} ${base_z_size/2}"/>
+          <mesh filename="package://sdvt_description/meshes/New Frame with car no wheels.stl" scale="0.03 0.03 0.03"/>
         </geometry>
       </collision>
@@ -74,14 +67,15 @@
 			</inertial>
 			<visual>
-				<origin xyz="0 0 0" rpy="0 0 0" />
+				<origin xyz="0 0 0" rpy="${M_PI/2} ${M_PI/2} 0" />
 				<geometry>
-					<!--<mesh filename="package://husky_description/meshes/wheel.dae" />-->
- 					<cylinder length="${wheel_length/4}" radius="${wheel_radius/4}" />
+					<!-- <mesh filename="package://sdvt_description/meshes/tire.stl" scale="0.03 0.03 0.03"/> -->
+ 					 <cylinder length="${wheel_length}" radius="${wheel_radius}" />
 				</geometry>
 			</visual>
 			<collision>
-				<origin xyz="0 0 0" rpy="${M_PI/2} 0 0" />
+				<origin xyz="0 0 0" rpy="${M_PI/2} ${M_PI/2} 0" />
 				<geometry>
-					<cylinder length="${wheel_length}" radius="${wheel_radius}" />
+					<!-- <mesh filename="package://sdvt_description/meshes/tire.stl" scale="0.03 0.03 0.03"/> -->
+ 					 <cylinder length="${wheel_length}" radius="${wheel_radius}" />
 				</geometry>
 			</collision>
@@ -139,9 +133,115 @@
     <origin xyz="-0.180 0.126 0.1815" />
   </joint>
+  <!-- Front radar -->
+<link name="Radar">
+    <visual>
+      <geometry>
+        <box size=".1 .23 .14"/>
+      </geometry>
+      <material name="white"/>
+      <origin xyz="0 0 0" rpy="0 0 0"/>
+    </visual>
+    <collision>
+      <geometry>
+        <box size=".1 .23 .14"/>
+      </geometry>
+    </collision>
+</link>
+ <joint name="base_to_radar" type="fixed">
+      <child link ="Radar" />
+      <parent link ="base_link" />
+      <origin xyz="3.2 0 0.4"/>
+      <axis>
+        <xyz>0 0 1</xyz>
+        <limit>
+          <upper>0</upper>
+          <lower>0</lower>
+        </limit>
+      </axis>
+    </joint>
   <!-- Left lidar -->
+  <link name="lidar_left">
+     <visual>
+       <origin xyz="0 0 0" rpy="0 0 0" />
+       <geometry>
+        <cylinder length="0.09" radius="0.05"/>
+      </geometry>
+      <material name="white"/>
+    </visual>
+  </link>
+    <joint name="hokuyo_joint_left" type="fixed">
+      <child link ="lidar_left" />
+      <parent link ="base_link" />
+      <origin xyz="-0.14 -1.72 0.42"/>
+      <axis>
+        <xyz>0 0 1</xyz>
+        <limit>
+          <upper>0</upper>
+          <lower>0</lower>
+        </limit>
+      </axis>
+    </joint>
   <!-- Right lidar -->
-  <!-- Front radar -->
+ <link name="lidar_right">
+     <visual>
+       <origin xyz="0 0 0" rpy="0 0 0" />
+       <geometry>
+        <cylinder length="0.09" radius="0.05"/>
+      </geometry>
+      <material name="white"/>
+    </visual>
+  </link>
+    <joint name="hokuyo_joint_right" type="fixed">
+      <child link ="lidar_right" />
+      <parent link ="base_link" />
+      <origin xyz="-0.14 1.72 0.42"/>
+      <axis>
+        <xyz>0 0 1</xyz>
+        <limit>
+          <upper>0</upper>
+          <lower>0</lower>
+        </limit>
+      </axis>
+    </joint>
   <!-- Left camera -->
+<link name="camera_l">
+    <visual>
+      <geometry>
+        <cylinder length="0.076" radius="0.04"/>
+      </geometry>
+      <material name="white"/>
+      <origin xyz="0 0 0" rpy="0 1.5708 0"/>
+    </visual>
+    <collision>
+      <geometry>
+        <cylinder length="0.05" radius="0.04"/>
+      </geometry>
+    </collision>
+</link>
+ <joint name="base_to_camera_l" type="fixed">
+      <child link ="camera_l" />
+      <parent link ="base_link" />
+      <origin xyz="1.5 -1.8 3"/>
+    </joint>
   <!-- Right camera -->
+   <link name="camera_r">
+    <visual>
+      <geometry>
+        <cylinder length="0.076" radius="0.04"/>
+      </geometry>
+      <material name="white"/>
+      <origin xyz="0 0 0" rpy="0 1.5708 0"/>
+    </visual>
+    <collision>
+      <geometry>
+        <cylinder length="0.05" radius="0.04"/>
+      </geometry>
+    </collision>
+</link>
+ <joint name="base_to_camera_r" type="fixed">
+      <child link ="camera_r" />
+      <parent link ="base_link" />
+      <origin xyz="1.5 1.8 3"/>
+    </joint>
   <xacro:include filename="sdvt.gazebo" />
 </robot>

Commit message: made some changes

File: src/sdvt_description/urdf/cart.urdf.xacro (robot description, xacro)
@@ -7,16 +7,16 @@
   <property name="base_z_size" value="1" />
   <!-- Wheel Mounting Positions -->
-  <xacro:property name="wheelbase" value="4.8" />
-  <xacro:property name="track" value="2.63" />
-  <xacro:property name="wheel_vertical_offset" value="-0.5" />
+  <xacro:property name="wheelbase" value="1.702" />
+  <xacro:property name="track" value="1.016" />
+  <xacro:property name="wheel_vertical_offset" value="-0.05" />
   <!-- Wheel Properties -->
-  <xacro:property name="wheel_length" value="1" />
-  <xacro:property name="wheel_radius" value="0.24" />
+  <xacro:property name="wheel_length" value="0.23" />
+  <xacro:property name="wheel_radius" value="0.242" />
     <!-- Base link is the center of the robot's bottom plate -->
     <link name="base_link">
       <visual>
-        <origin xyz="0 1.65 0" rpy="${M_PI/2} 0 0" />
+        <origin xyz="0 0.559 0" rpy="${M_PI/2} 0 0" />
         <geometry>
-          <mesh filename="package://sdvt_description/meshes/New Frame with car no wheels.stl" scale="0.03 0.03 0.03"/>
+          <mesh filename="package://sdvt_description/meshes/New Frame with car no wheels meters.stl" scale="0.0104 0.0104 0.0104"/>
         </geometry>
       </visual>
@@ -24,5 +24,5 @@
         <origin xyz="0 0 ${base_z_size/4}" rpy="0 0 0" />
         <geometry>
-          <mesh filename="package://sdvt_description/meshes/New Frame with car no wheels.stl" scale="0.03 0.03 0.03"/>
+          <mesh filename="package://sdvt_description/meshes/New Frame with car no wheels meters.stl" scale="0.0104 0.0104 0.0104"/>
         </geometry>
       </collision>
@@ -69,6 +69,6 @@
 				<origin xyz="0 0 0" rpy="${M_PI/2} ${M_PI/2} 0" />
 				<geometry>
-					<!-- <mesh filename="package://sdvt_description/meshes/tire.stl" scale="0.03 0.03 0.03"/> -->
- 					 <cylinder length="${wheel_length}" radius="${wheel_radius}" />
+					 <mesh filename="package://sdvt_description/meshes/tire meters.stl" scale="0.104 0.104 0.104"/>
+ 					 <!--<cylinder length="${wheel_length}" radius="${wheel_radius}" /> -->
 				</geometry>
 			</visual>
@@ -76,6 +76,6 @@
 				<origin xyz="0 0 0" rpy="${M_PI/2} ${M_PI/2} 0" />
 				<geometry>
-					<!-- <mesh filename="package://sdvt_description/meshes/tire.stl" scale="0.03 0.03 0.03"/> -->
- 					 <cylinder length="${wheel_length}" radius="${wheel_radius}" />
+					 <mesh filename="package://sdvt_description/meshes/tire meters.stl" scale="0.0104 0.0104 0.0104"/>
+ 					<!-- <cylinder length="${wheel_length}" radius="${wheel_radius}" />-->
 				</geometry>
 			</collision>
@@ -151,5 +151,5 @@
       <child link ="Radar" />
       <parent link ="base_link" />
-      <origin xyz="3.2 0 0.4"/>
+      <origin xyz="1.18 0 0.2"/>
       <axis>
         <xyz>0 0 1</xyz>
@@ -161,5 +161,12 @@
     </joint>
   <!-- Left lidar -->
-  <link name="lidar_left">
+  <link name="lidar_left_link">
+<!--<inertial>
+      <mass value="0.01" />
+      <origin xyz="0 0 0" />
+      <inertia ixx="0.001"  ixy="0.0"  ixz="0.0"
+               iyy="0.001"  iyz="0.0"
+               izz="0.001" />
+    </inertial> -->
      <visual>
        <origin xyz="0 0 0" rpy="0 0 0" />
@@ -171,7 +178,7 @@
   </link>
     <joint name="hokuyo_joint_left" type="fixed">
-      <child link ="lidar_left" />
-      <parent link ="base_link" />
-      <origin xyz="-0.14 -1.72 0.42"/>
+      <child link ="lidar_left_link" />
+      <parent link ="base_link" />
+      <origin xyz="-0.11 -0.65 0.12"/>
       <axis>
         <xyz>0 0 1</xyz>
@@ -195,5 +202,5 @@
       <child link ="lidar_right" />
       <parent link ="base_link" />
-      <origin xyz="-0.14 1.72 0.42"/>
+      <origin xyz="-0.11 0.65 0.12"/>
       <axis>
         <xyz>0 0 1</xyz>
@@ -222,5 +229,5 @@
       <child link ="camera_l" />
       <parent link ="base_link" />
-      <origin xyz="1.5 -1.8 3"/>
+      <origin xyz="0.5 -0.65 1.1"/>
     </joint>
   <!-- Right camera -->
@@ -242,5 +249,5 @@
       <child link ="camera_r" />
       <parent link ="base_link" />
-      <origin xyz="1.5 1.8 3"/>
+      <origin xyz="0.5 0.6 1.1"/>
     </joint>
   <xacro:include filename="sdvt.gazebo" />

Commit message: update files

File: src/sdvt_description/urdf/cart.urdf.xacro (robot description, xacro)
@@ -1,5 +1,5 @@
 <?xml version="1.0"?>
 <robot name="sdvt_robot" xmlns:xacro="http://ros.org/wiki/xacro">
-  <property name="M_PI" value="3.14159"/>
+  <property name="M_PI" value="3.1415926535897931"/>
   <!-- Base Size -->
   <property name="base_x_size" value="3" />
@@ -18,11 +18,14 @@
         <origin xyz="0 0.559 0" rpy="${M_PI/2} 0 0" />
         <geometry>
-          <mesh filename="package://sdvt_description/meshes/New Frame with car no wheels meters.stl" scale="0.0104 0.0104 0.0104"/>
+          <mesh filename="package://sdvt_description/meshes/Frame.stl" scale="0.0104 0.0104 0.0104"/>
         </geometry>
+        <material name="grey">
+          <color rgba=".748 .748 .755 1"/>
+        </material>
       </visual>
       <collision>
-        <origin xyz="0 0 ${base_z_size/4}" rpy="0 0 0" />
+        <origin xyz="0 0.559 0" rpy="${M_PI/2} 0 0" />
         <geometry>
-          <mesh filename="package://sdvt_description/meshes/New Frame with car no wheels meters.stl" scale="0.0104 0.0104 0.0104"/>
+          <mesh filename="package://sdvt_description/meshes/Frame.stl" scale="0.0104 0.0104 0.0104"/>
         </geometry>
       </collision>
@@ -38,7 +41,7 @@
     <link name="inertial_link">
       <inertial>
-        <mass value="33.455" />
-        <origin xyz="-0.08748 -0.00085 0.09947" />
-        <inertia ixx="0.6022" ixy="-0.02364" ixz="-0.1197" iyy="1.7386" iyz="-0.001544" izz="2.0296" />
+        <mass value="125" />
+        <origin xyz="0 0 0" />
+        <inertia ixx="1.391" ixy="0.004"  ixz="0.0"  iyy="6.853"  iyz="0.0"  izz="6.125" />
       </inertial>
     </link>
@@ -58,5 +61,5 @@
     <gazebo reference="imu_link">
     </gazebo>
-    <!-- SDVT wheel xacro -->
+  <!-- SDVT wheel xacro -->
 	<xacro:macro name="sdvt_wheel" params="wheel_prefix *joint_pose">
 		<link name="${wheel_prefix}_wheel_link">
@@ -67,15 +70,18 @@
 			</inertial>
 			<visual>
-				<origin xyz="0 0 0" rpy="${M_PI/2} ${M_PI/2} 0" />
+				<origin xyz="0 0.089 0" rpy="${M_PI/2} ${M_PI/2} 0" />
 				<geometry>
-					 <mesh filename="package://sdvt_description/meshes/tire meters.stl" scale="0.104 0.104 0.104"/>
- 					 <!--<cylinder length="${wheel_length}" radius="${wheel_radius}" /> -->
+					 <!--<mesh filename="package://sdvt_description/meshes/tire.stl" scale="0.0104 0.0104 0.0104"/>-->
+ 					 <cylinder length="${wheel_length}" radius="${wheel_radius}" />
 				</geometry>
+        <material name="grey">
+          <color rgba=".13 .13 .13 1"/>
+        </material>
 			</visual>
 			<collision>
-				<origin xyz="0 0 0" rpy="${M_PI/2} ${M_PI/2} 0" />
+				<origin xyz="0 0.089 0" rpy="${M_PI/2} ${M_PI/2} 0" />
 				<geometry>
-					 <mesh filename="package://sdvt_description/meshes/tire meters.stl" scale="0.0104 0.0104 0.0104"/>
- 					<!-- <cylinder length="${wheel_length}" radius="${wheel_radius}" />-->
+					 <!-- <mesh filename="package://sdvt_description/meshes/tire.stl" scale="0.0104 0.0104 0.0104"/> -->
+ 					 <cylinder length="${wheel_length}" radius="${wheel_radius}" />
 				</geometry>
 			</collision>
@@ -133,5 +139,5 @@
     <origin xyz="-0.180 0.126 0.1815" />
   </joint>
-  <!-- Front radar -->
+<!-- Front radar -->
 <link name="Radar">
     <visual>
@@ -147,5 +153,10 @@
       </geometry>
     </collision>
-</link>
+    <inertial>
+      <mass value="0.01"/>
+      <origin xyz="0 0 0"/>
+      <inertia ixx="0.0001" ixy="0.0" ixz="0.0" iyy="0.0001" iyz="0.0" izz="0.0001"/>
+    </inertial>
+ </link>
  <joint name="base_to_radar" type="fixed">
       <child link ="Radar" />
@@ -161,24 +172,32 @@
     </joint>
   <!-- Left lidar -->
+  <xacro:include filename="$(find sdvt_description)/urdf/sensors/hokuyo_laser.urdf.xacro"/>
+	<xacro:hokuyo_laser name="left_laser" parent="lidar_left" ros_topic="/scan" update_rate="20" min_angle="-1.57" max_angle="1.57">
+		<origin xyz="0 0 0" rpy="0 0 0" />
+	</xacro:hokuyo_laser>
   <link name="lidar_left_link">
-<!--<inertial>
-      <mass value="0.01" />
-      <origin xyz="0 0 0" />
-      <inertia ixx="0.001"  ixy="0.0"  ixz="0.0"
-               iyy="0.001"  iyz="0.0"
-               izz="0.001" />
-    </inertial> -->
-     <visual>
+    <visual>
+      <origin xyz="0 0 0" rpy="0 0 0" />
+       <geometry>
+        <cylinder length="0.09" radius="0.05"/>
+      </geometry>
+      <material name="white"/>
+    </visual>
+    <collision>
        <origin xyz="0 0 0" rpy="0 0 0" />
        <geometry>
         <cylinder length="0.09" radius="0.05"/>
       </geometry>
-      <material name="white"/>
-    </visual>
-  </link>
-    <joint name="hokuyo_joint_left" type="fixed">
+    </collision>
+    <inertial>
+      <mass value="1e-5" />
+      <origin xyz="0 0 0" rpy="0 0 0"/>
+      <inertia ixx="1e-6" ixy="0" ixz="0" iyy="1e-6" iyz="0" izz="1e-6" />
+    </inertial>
+  </link>
+    <joint name="hokuyo_left_joint" type="fixed">
       <child link ="lidar_left_link" />
       <parent link ="base_link" />
-      <origin xyz="-0.11 -0.65 0.12"/>
+      <origin xyz="-0.11 -0.65 0.12" rpy="0 0 -1.57"/>
       <axis>
         <xyz>0 0 1</xyz>
@@ -190,5 +209,8 @@
     </joint>
   <!-- Right lidar -->
- <link name="lidar_right">
+	<xacro:hokuyo_laser name="right_laser" parent="lidar_right" ros_topic="/scan" update_rate="20" min_angle="-1.57" max_angle="1.57">
+		<origin xyz="0 0 0" rpy="0 0 0" />
+	</xacro:hokuyo_laser>
+ <link name="lidar_right_link">
      <visual>
        <origin xyz="0 0 0" rpy="0 0 0" />
@@ -198,9 +220,20 @@
       <material name="white"/>
     </visual>
-  </link>
-    <joint name="hokuyo_joint_right" type="fixed">
-      <child link ="lidar_right" />
-      <parent link ="base_link" />
-      <origin xyz="-0.11 0.65 0.12"/>
+    <collision>
+       <origin xyz="0 0 0" rpy="0 0 0" />
+       <geometry>
+        <cylinder length="0.09" radius="0.05"/>
+      </geometry>
+    </collision>
+    <inertial>
+      <mass value="1e-5" />
+      <origin xyz="0 0 0" rpy="0 0 0"/>
+      <inertia ixx="1e-6" ixy="0" ixz="0" iyy="1e-6" iyz="0" izz="1e-6" />
+    </inertial>
+  </link>
+    <joint name="hokuyo_right_joint" type="fixed">
+      <child link ="lidar_right_link" />
+      <parent link ="base_link" />
+      <origin xyz="-0.11 0.6 0.12" rpy="0 0 1.57"/>
       <axis>
         <xyz>0 0 1</xyz>
@@ -222,5 +255,5 @@
     <collision>
       <geometry>
-        <cylinder length="0.05" radius="0.04"/>
+        <cylinder length="0.076" radius="0.04"/>
       </geometry>
     </collision>
@@ -242,13 +275,13 @@
     <collision>
       <geometry>
-        <cylinder length="0.05" radius="0.04"/>
-      </geometry>
-    </collision>
-</link>
- <joint name="base_to_camera_r" type="fixed">
+        <cylinder length="0.076" radius="0.04"/>
+      </geometry>
+    </collision>
+  </link>
+  <joint name="base_to_camera_r" type="fixed">
       <child link ="camera_r" />
       <parent link ="base_link" />
       <origin xyz="0.5 0.6 1.1"/>
     </joint>
-  <xacro:include filename="sdvt.gazebo" />
+  <xacro:include filename="$(find sdvt_description)/urdf/sdvt.gazebo" />
 </robot>
