Commit message: Updated footer

File: src/sdvt_description/urdf/cart.urdf.xacro (robot description, xacro)
@@ -1,5 +1,6 @@
 <?xml version="1.0"?>
 <robot name="sdvt_robot" xmlns:xacro="http://ros.org/wiki/xacro">
-  <property name="M_PI" value="3.1415926535897931"/>
+  <xacro:include filename="$(find sdvt_description)/urdf/wheel.urdf.xacro" />
+  <property name="M_PI" value="3.14159"/>
   <!-- Base Size -->
   <property name="base_x_size" value="3" />
@@ -20,7 +21,7 @@
           <mesh filename="package://sdvt_description/meshes/Frame.stl" scale="0.0104 0.0104 0.0104"/>
         </geometry>
-        <material name="grey">
-          <color rgba=".748 .748 .755 1"/>
-        </material>
+      <material name="grey">
+        <color rgba=".748 .748 .755 1"/>
+      </material>
       </visual>
       <collision>
@@ -34,14 +35,29 @@
     <link name="base_footprint"/>
     <joint name="base_footprint_joint" type="fixed">
-      <origin xyz="0 0 ${wheel_vertical_offset - wheel_radius}" rpy="0 0 0" />
-      <parent link="base_link" />
-      <child link="base_footprint" />
-    </joint>
+      <origin xyz="0 0 ${-wheel_vertical_offset + wheel_radius}" rpy="0 0 0" />
+      <parent link="base_footprint" />
+      <child link="base_link" />
+    </joint>
+<!-- Navsat link -->
+	  <link name="navsat_link">
+		<visual>
+		  <geometry>
+		    <cylinder radius="0.026" length="0.016" />
+		  </geometry>
+		  <origin xyz="0 0 0" />
+		  <material name="black" />
+		</visual>
+	  </link>
+	  <joint name="navsat_joint" type="fixed">
+		<parent link="base_link" />
+		<child link="navsat_link" />
+		<origin xyz="0 0 0" />
+	  </joint>
     <!-- Interial link stores the robot's inertial information -->
     <link name="inertial_link">
       <inertial>
-        <mass value="125" />
-        <origin xyz="0 0 0" />
-        <inertia ixx="1.391" ixy="0.004"  ixz="0.0"  iyy="6.853"  iyz="0.0"  izz="6.125" />
+        <mass value="33.455" />
+        <origin xyz="-0.08748 -0.00085 0.09947" />
+        <inertia ixx="0.6022" ixy="-0.02364" ixz="-0.1197" iyy="1.7386" iyz="-0.001544" izz="2.0296" />
       </inertial>
     </link>
@@ -61,54 +77,5 @@
     <gazebo reference="imu_link">
     </gazebo>
-  <!-- SDVT wheel xacro -->
-	<xacro:macro name="sdvt_wheel" params="wheel_prefix *joint_pose">
-		<link name="${wheel_prefix}_wheel_link">
-			<inertial>
-				<mass value="2.637" />
-				<origin xyz="0 0 0" />
-				<inertia  ixx="0.02467" ixy="0" ixz="0" iyy="0.02467" iyz="0" izz="0.04411" />
-			</inertial>
-			<visual>
-				<origin xyz="0 0.089 0" rpy="${M_PI/2} ${M_PI/2} 0" />
-				<geometry>
-					 <!--<mesh filename="package://sdvt_description/meshes/tire.stl" scale="0.0104 0.0104 0.0104"/>-->
- 					 <cylinder length="${wheel_length}" radius="${wheel_radius}" />
-				</geometry>
-        <material name="grey">
-          <color rgba=".13 .13 .13 1"/>
-        </material>
-			</visual>
-			<collision>
-				<origin xyz="0 0.089 0" rpy="${M_PI/2} ${M_PI/2} 0" />
-				<geometry>
-					 <!-- <mesh filename="package://sdvt_description/meshes/tire.stl" scale="0.0104 0.0104 0.0104"/> -->
- 					 <cylinder length="${wheel_length}" radius="${wheel_radius}" />
-				</geometry>
-			</collision>
-		</link>
-		<gazebo reference="${wheel_prefix}_wheel_link">
-			<mu1 value="1.0"/>
-			<mu2 value="1.0"/>
-			<kp value="10000000.0" />
-			<kd value="1.0" />
-			<fdir1 value="1 0 0"/>
-		</gazebo>
-		<joint name="${wheel_prefix}_wheel" type="continuous">
-			<parent link="base_link"/>
-			<child link="${wheel_prefix}_wheel_link"/>
-			<xacro:insert_block name="joint_pose"/>
-			<axis xyz="0 1 0" rpy="0 0 0" />
-		</joint>
-		<transmission name="${wheel_prefix}_wheel_trans" type="SimpleTransmission">
-			<type>transmission_interface/SimpleTransmission</type>
-			<actuator name="${wheel_prefix}_wheel_motor">
-				<mechanicalReduction>1</mechanicalReduction>
-			</actuator>
-			<joint name="${wheel_prefix}_wheel">
-				<hardwareInterface>VelocityJointInterface</hardwareInterface>
-			</joint>
-		</transmission>
-	</xacro:macro>
-    <!-- SDVT wheel macros -->
+    <!-- SDVT wheel macros
     <xacro:sdvt_wheel wheel_prefix="front_left">
       <origin xyz="${wheelbase/2} ${track/2} ${wheel_vertical_offset}" rpy="0 0 0" />
@@ -122,11 +89,23 @@
     <xacro:sdvt_wheel wheel_prefix="rear_right">
       <origin xyz="${-wheelbase/2} ${-track/2} ${wheel_vertical_offset}" rpy="0 0 0" />
-    </xacro:sdvt_wheel>
-  <!-- Decoration description  <xacro:sdvt_decorate /> -->
+    </xacro:sdvt_wheel>-->
+    <!-- SDVT wheel ARKMEN macros -->
+    <xacro:front_wheel lr_prefix="left" fr_prefix="front" lr_reflect="1" fr_reflect="1">
+      <origin xyz="${wheelbase/2} ${track/2} ${wheel_vertical_offset}" rpy="0 0 0" />
+    </xacro:front_wheel>
+    <xacro:front_wheel lr_prefix="right" fr_prefix="front" lr_reflect="-1" fr_reflect="1">
+      <origin xyz="${wheelbase/2} ${-track/2} ${wheel_vertical_offset}" rpy="0 0 0" />
+    </xacro:front_wheel>
+    <xacro:rear_wheel lr_prefix="left" fr_prefix="rear" lr_reflect="1" fr_reflect="-1">
+      <origin xyz="${-wheelbase/2} ${track/2} ${wheel_vertical_offset}" rpy="0 0 0" />
+    </xacro:rear_wheel>
+    <xacro:rear_wheel lr_prefix="right" fr_prefix="rear" lr_reflect="-1" fr_reflect="-1">
+      <origin xyz="${-wheelbase/2} ${-track/2} ${wheel_vertical_offset}" rpy="0 0 0" />
+    </xacro:rear_wheel>
   <!-- Same note as applies to imu_link -->
-  <link name="navsat_link">
-    <visual>
-      <geometry>
-        <cylinder radius="0.026" length="0.016" />
+  <link name="GPS_link">
+    <visual>
+      <geometry>
+        <box size="0.1 0.1 0.05" />
       </geometry>
       <origin xyz="0 0 0.008" />
@@ -134,14 +113,14 @@
     </visual>
   </link>
-  <joint name="navsat_joint" type="fixed">
+  <joint name="gps_joint" type="fixed">
     <parent link="base_link" />
-    <child link="navsat_link" />
-    <origin xyz="-0.180 0.126 0.1815" />
+    <child link="GPS_link" />
+    <origin xyz="0 0 0.54" />
   </joint>
-<!-- Front radar -->
-<link name="Radar">
-    <visual>
-      <geometry>
-        <box size=".1 .23 .14"/>
+  <!-- Front radar -->
+<link name="Lidar">
+    <visual>
+      <geometry>
+        <box size=".1 .18 .11"/>
       </geometry>
       <material name="white"/>
@@ -160,5 +139,5 @@
  </link>
  <joint name="base_to_radar" type="fixed">
-      <child link ="Radar" />
+      <child link ="Lidar" />
       <parent link ="base_link" />
       <origin xyz="1.18 0 0.2"/>
@@ -172,9 +151,5 @@
     </joint>
   <!-- Left lidar -->
-  <xacro:include filename="$(find sdvt_description)/urdf/sensors/hokuyo_laser.urdf.xacro"/>
-	<xacro:hokuyo_laser name="left_laser" parent="lidar_left" ros_topic="/scan" update_rate="20" min_angle="-1.57" max_angle="1.57">
-		<origin xyz="0 0 0" rpy="0 0 0" />
-	</xacro:hokuyo_laser>
-  <link name="lidar_left_link">
+  <link name="lidar_left">
     <visual>
       <origin xyz="0 0 0" rpy="0 0 0" />
@@ -196,6 +171,6 @@
     </inertial>
   </link>
-    <joint name="hokuyo_left_joint" type="fixed">
-      <child link ="lidar_left_link" />
+    <joint name="hokuyo_joint_left" type="fixed">
+      <child link ="lidar_left" />
       <parent link ="base_link" />
       <origin xyz="-0.11 -0.65 0.12" rpy="0 0 -1.57"/>
@@ -209,8 +184,5 @@
     </joint>
   <!-- Right lidar -->
-	<xacro:hokuyo_laser name="right_laser" parent="lidar_right" ros_topic="/scan" update_rate="20" min_angle="-1.57" max_angle="1.57">
-		<origin xyz="0 0 0" rpy="0 0 0" />
-	</xacro:hokuyo_laser>
- <link name="lidar_right_link">
+ <link name="lidar_right">
      <visual>
        <origin xyz="0 0 0" rpy="0 0 0" />
@@ -232,6 +204,6 @@
     </inertial>
   </link>
-    <joint name="hokuyo_right_joint" type="fixed">
-      <child link ="lidar_right_link" />
+    <joint name="hokuyo_joint_right" type="fixed">
+      <child link ="lidar_right" />
       <parent link ="base_link" />
       <origin xyz="-0.11 0.6 0.12" rpy="0 0 1.57"/>
@@ -262,5 +234,5 @@
       <child link ="camera_l" />
       <parent link ="base_link" />
-      <origin xyz="0.5 -0.65 1.1"/>
+      <origin xyz="0.5 -0.65 1.6" rpy="3.141 0 0"/>
     </joint>
   <!-- Right camera -->
@@ -282,6 +254,64 @@
       <child link ="camera_r" />
       <parent link ="base_link" />
-      <origin xyz="0.5 0.6 1.1"/>
-    </joint>
-  <xacro:include filename="$(find sdvt_description)/urdf/sdvt.gazebo" />
+      <origin xyz="0.5 0.6 1.6" rpy="3.141 0 0"/>
+    </joint>
+<!-- Added side and back camera -->
+    <link name="camera_side_right">
+    <visual>
+      <geometry>
+        <cylinder length="0.076" radius="0.04"/>
+      </geometry>
+      <material name="white"/>
+      <origin xyz="0 0 0" rpy="0 1.5708 0"/>
+    </visual>
+    <collision>
+      <geometry>
+        <cylinder length="0.076" radius="0.04"/>
+      </geometry>
+    </collision>
+  </link>
+  <joint name="base_to_camera_side_right" type="fixed">
+      <child link ="camera_side_right" />
+      <parent link ="base_link" />
+      <origin xyz="-0.62 0.6 1.6" rpy="0 0 1.5708"/>
+    </joint>
+  <link name="camera_side_left">
+    <visual>
+      <geometry>
+        <cylinder length="0.076" radius="0.04"/>
+      </geometry>
+      <material name="white"/>
+      <origin xyz="0 0 0" rpy="0 1.5708 0"/>
+    </visual>
+    <collision>
+      <geometry>
+        <cylinder length="0.076" radius="0.04"/>
+      </geometry>
+    </collision>
+  </link>
+  <joint name="base_to_camera_side_left" type="fixed">
+      <child link ="camera_side_left" />
+      <parent link ="base_link" />
+      <origin xyz="-0.62 -0.65 1.6" rpy="0 0 -1.5708"/>
+    </joint>
+  <link name="camera_back">
+    <visual>
+      <geometry>
+        <cylinder length="0.076" radius="0.04"/>
+      </geometry>
+      <material name="white"/>
+      <origin xyz="0 0 0" rpy="0 1.5708 0"/>
+    </visual>
+    <collision>
+      <geometry>
+        <cylinder length="0.076" radius="0.04"/>
+      </geometry>
+    </collision>
+   </link>
+   <joint name="base_to_camera_back" type="fixed">
+      <child link ="camera_back" />
+      <parent link ="base_link" />
+      <origin xyz="-0.7 0 1.6" rpy="0 0 3.1416"/>
+    </joint>
+  <xacro:include filename="sdvt.gazebo" />
 </robot>

File: src/sdvt_description/urdf/wheel.urdf.xacro (robot description, xacro)
@@ -1,5 +1,5 @@
 <?xml version="1.0"?>
 <robot xmlns:xacro="http://ros.org/wiki/xacro" name="sdvt_wheel">
-	<xacro:macro name="sdvt_wheel" params="wheel_prefix *joint_pose">
+	<!--<xacro:macro name="sdvt_wheel" params="wheel_prefix *joint_pose">
 		<link name="${wheel_prefix}_wheel_link">
 			<inertial>
@@ -11,5 +11,4 @@
 				<origin xyz="0 0 0" rpy="0 0 0" />
 				<geometry>
-					<!--<mesh filename="package://husky_description/meshes/wheel.dae" />-->
  					<cylinder length="${wheel_length}" radius="${wheel_radius}" />
 				</geometry>
@@ -44,4 +43,128 @@
 			</joint>
 		</transmission>
+	</xacro:macro>-->
+  <xacro:property name="wheel_joint_damping" value="0.2" />
+  <xacro:property name="wheel_joint_friction" value="0.7" />
+  <xacro:property name="axle_eff_limit" value="204.95"/>
+  <xacro:property name="axle_vel_limit" value="39.02"/>
+  <xacro:property name="servo_stall_torque" value="50"/>  <!-- check -->
+  <xacro:property name="servo_no_load_speed" value="25"/> <!-- check -->
+  <!-- Wheel Mounting Positions -->
+  <xacro:property name="wheelbase" value="1.702" />
+  <xacro:property name="track" value="1.016" />
+  <xacro:property name="wheel_vertical_offset" value="-0.05" />
+  <!-- Degree-to-radian conversions -->
+  <xacro:property name="degrees_45" value="0.785398163"/>
+  <xacro:property name="degrees_90" value="1.57079633"/>
+  <xacro:property name="degrees_180" value="3.14159265"/>
+  <!-- Null inertial element. This is needed to make the model work with
+       Gazebo. -->
+  <xacro:macro name="null_inertial">
+    <inertial>
+      <mass value="0.001"/>
+      <inertia ixx="0.001" ixy="0" ixz="0" iyy="0.001" iyz="0" izz="0.001"/>
+    </inertial>
+  </xacro:macro>
+  <!-- The "wheel" macro defines an axle carrier, axle, and wheel. -->
+  <xacro:macro name="wheel" params="lr_prefix fr_prefix lr_reflect fr_reflect ">
+    <link name="${lr_prefix}_${fr_prefix}_axle_carrier">
+      <xacro:null_inertial/>
+    </link>
+    <link name="${lr_prefix}_${fr_prefix}_wheel">
+			<inertial>
+				<mass value="2.637" />
+				<origin xyz="0 0 0" />
+				<inertia  ixx="0.02467" ixy="0" ixz="0" iyy="0.02467" iyz="0" izz="0.04411" />
+			</inertial>
+			<visual>
+				<origin xyz="0 0 0" rpy="0 0 0" />
+				<geometry>
+ 					<cylinder length="${wheel_length}" radius="${wheel_radius}" />
+				</geometry>
+			</visual>
+			<collision>
+				<origin xyz="0 0 0" rpy="${M_PI/2} 0 0" />
+				<geometry>
+					<cylinder length="${wheel_length}" radius="${wheel_radius}" />
+				</geometry>
+			</collision>
+	</link>
+    <!-- The left and right axles have the same axis so that identical
+         rotation values cause the wheels to rotate in the same direction. -->
+    <joint name="${lr_prefix}_${fr_prefix}_axle" type="continuous">
+      <parent link="${lr_prefix}_${fr_prefix}_axle_carrier"/>
+      <child link="${lr_prefix}_${fr_prefix}_wheel"/>
+	  <axis xyz="0 0 1" rpy="0 0 0" />
+      <origin rpy="${degrees_90} 0 ${degrees_180}"/>
+      <limit effort="${axle_eff_limit}" velocity="${axle_vel_limit}"/>
+      <joint_properties damping="${wheel_joint_damping}" friction="{wheel_joint_friction}"/>
+    </joint>
+    <transmission name="${lr_prefix}_${fr_prefix}_axle_trans">
+      <type>transmission_interface/SimpleTransmission</type>
+      <joint name="${lr_prefix}_${fr_prefix}_axle">
+        <hardwareInterface>VelocityJointInterface</hardwareInterface>
+      </joint>
+      <actuator name="${lr_prefix}_${fr_prefix}_axle_act">
+        <mechanicalReduction>1</mechanicalReduction>
+      </actuator>
+    </transmission>
+    <gazebo reference="${lr_prefix}_${fr_prefix}_axle_carrier">
+      <material>Gazebo/Black</material>
+    </gazebo>
+    <gazebo reference="${lr_prefix}_${fr_prefix}_wheel">
+      <material>Gazebo/Black</material>
+    </gazebo>
+  </xacro:macro>
+	<!-- Front wheel -->
+	<xacro:macro name="front_wheel" params="lr_prefix fr_prefix lr_reflect fr_reflect *joint_pose">
+		<link name="${lr_prefix}_steering_link">
+			<xacro:null_inertial/>
+    	</link>
+		<joint name="${lr_prefix}_front_base" type="fixed">
+			<parent link="base_link"/>
+			<child link="${lr_prefix}_steering_link"/>
+			<axis xyz="0 0 1" rpy="0 0 0" />
+		</joint>
+		<joint name="${lr_prefix}_steering_joint" type="revolute">
+			<parent link="base_link"/>
+			<child link="${lr_prefix}_${fr_prefix}_axle_carrier"/>
+			<xacro:insert_block name="joint_pose"/>
+			<axis xyz="0 1 0" rpy="0 0 0" />
+			<limit lower="${-degrees_45}" upper="${degrees_45}" effort="${servo_stall_torque}" velocity="${servo_no_load_speed}"/>
+		</joint>
+		<transmission name="${lr_prefix}_steering_trans">
+			<type>transmission_interface/SimpleTransmission</type>
+			<joint name="${lr_prefix}_steering_joint">
+				<hardwareInterface>EffortJointInterface</hardwareInterface>
+			</joint>
+			<actuator name="${lr_prefix}_steering_act">
+				<mechanicalReduction>1</mechanicalReduction>
+			</actuator>
+		</transmission>
+		<!--<gazebo reference="${lr_prefix}_steering_link">
+			<material>Gazebo/Black</material>
+		</gazebo>-->
+    	<xacro:wheel lr_prefix="${lr_prefix}" fr_prefix="${fr_prefix}" lr_reflect="${lr_reflect}" fr_reflect="${fr_reflect}"/>
+	</xacro:macro>
+	<!-- Rear wheel -->
+	<xacro:macro name="rear_wheel" params="lr_prefix fr_prefix lr_reflect fr_reflect *joint_pose">
+		<link name="${lr_prefix}_rear_link">
+			<xacro:null_inertial/>
+    	</link>
+		<joint name="${lr_prefix}_rear_base" type="fixed">
+			<parent link="base_link"/>
+			<child link="${lr_prefix}_rear_link"/>
+			<axis xyz="0 0 1" rpy="0 0 0" />
+		</joint>
+		<joint name="${lr_prefix}_rear_joint" type="fixed">
+			<parent link="base_link"/>
+			<child link="${lr_prefix}_${fr_prefix}_axle_carrier"/>
+			<xacro:insert_block name="joint_pose"/>
+			<axis xyz="0 0 1" rpy="0 0 0" />
+		</joint>
+		<!--<gazebo reference="${lr_prefix}_rear_link">
+			<material>Gazebo/Black</material>
+		</gazebo>-->
+	<xacro:wheel lr_prefix="${lr_prefix}" fr_prefix="${fr_prefix}" lr_reflect="${lr_reflect}" fr_reflect="${fr_reflect}"/>
 	</xacro:macro>
 </robot>
